File: V1.7/ASSY_1_7/PlayerFront_1_7/PlayerFront02.kicad_pcb (KiCad board)
At the start: 2 copper layers, 165 x 51.5 mm, 18 parts, among them J2 Conn_01x04, J3 Conn_01x04, J4 AFC11-S30ICA-00

Commit message: Adjusted mounting holes
Made mounting holes a bit oval, to enable tiny positional adjustments.
Parts:
- H10, H11, H12, H9: footprint MountingHole:MountingHole_3.5mm -> !Gloeidraad:MountingSlot_3.5x4.0mm
