File: V1.7/ASSY_1_7/PlayerFront_1_7/PlayerFront02.kicad_sch (KiCad schematic)
At the start: 18 parts, among them J2 Conn_01x04, J3 Conn_01x04, J4 AFC11-S30ICA-00

Commit message: Add files via upload
Parts:
- H10, H9: footprint MountingHole:MountingHole_3.5mm -> !Gloeidraad:MountingSlot_3.5x4.0mm
Changed lines of the file:
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@@
 			)
 		)
-		(property "Footprint" "MountingHole:MountingHole_3.5mm"
+		(property "Footprint" "!Gloeidraad:MountingSlot_3.5x4.0mm"
 			(at 149.86 151.13 0)
 			(effects
@@
 			)
 		)
-		(property "Footprint" "MountingHole:MountingHole_3.5mm"
+		(property "Footprint" "!Gloeidraad:MountingSlot_3.5x4.0mm"
 			(at 135.89 151.13 0)
 			(effects
